Commit message: Edited Params

File: src/abhiyan_description/urdf/abhiyan.urdf (robot description, URDF)
Before this commit: robot abhiyan, 5 links, 4 joints
Joints:
- joint bot_base_camera_base: origin xyz=0 10 0 rpy=0 0 0 -> xyz=0 1.5 0 rpy=0 0 0
- joint bot_base_lidar: origin xyz=0 5 0 rpy=0 0 0 -> xyz=0 1 0 rpy=0 0 0

Commit message: Updates after a long time

File: src/abhiyan_description/urdf/abhiyan.urdf (robot description, URDF)
Before this commit: robot abhiyan, 5 links, 4 joints
Joints:
- joint bot_base_lidar: origin xyz=0 1 0 rpy=0 0 0 -> xyz=0.30 0 0 rpy=0 0 0
